File: circuits/driver-board.sch (KiCad schematic (older format))
At the start: 55 parts, among them J1 Motor_Conn_01x04, J2 Power_In_Conn_01x02, SW1 ESP_EN_SW_Push, SW2 ESP_IO0_SW_Push, U1 ESP32-WROOM-32U, U2 AS5601-ASOT, U3 TMC2209-LA, U5 MP2360DG-LF

Commit message: Fixed references with external KiCAD library
Parts:
- removed U3: TMC2209-LA, Package_DFN_QFN:QFN-28-1EP_5x5mm_P0.5mm_EP3.35x3.35mm_ThermalVias, symbol Driver_Motor_Local:TMC2209-LA
- added U5: TMC2209-LA, Package_DFN_QFN:QFN-28-1EP_5x5mm_P0.5mm_EP3.35x3.35mm_ThermalVias, symbol Slimc_Driver_Motor:TMC2209-LA
- U2: renamed from U5; symbol Regulator_Switching_Local:MP2360DG-LF -> Slimc_Regulator_Switching:MP2360DG-LF
- U4: renamed from U2; footprint Package_SO:SOIC-8_3.9x4.9mm_P1.27mm -> Package_DFN_QFN:QFN-24-1EP_4x4mm_P0.5mm_EP2.6x2.6mm; symbol Sensor_Magnetic_Local:AS5601-ASOT -> Slimc_Sensor_Magnetic:AS5601-ASOT
- gave numbers to parts that had none: 2
- renumbered C4 to C10, C5 to C11, C8 to C12, C15 to C13, C16 to C14, C17 to C15, C18 to C16, C19 to C17, C6 to C18, C9 to C19, C12 to C2, C22 to C20, C20 to C21, C21 to C22, C10 to C3, C14 to C4, C3 to C5, C2 to C6, C11 to C7, C13 to C8, C7 to C9, J1 to J3, R14 to R10, R3 to R11, R9 to R12, R10 to R13, R5 to R14, R11 to R2, R12 to R3, R13 to R4, R15 to R5, R16 to R6, R17 to R7, R18 to R8, R19 to R9, U1 to U3

Commit message: Work on schematics
Parts:
- removed C20: 330µF-50V, Capacitor_SMD:CP_Elec_5x3, symbol Device:CP_Small
- removed C5: 100µF, Capacitor_SMD:C_1206_3216Metric, symbol Device:CP_Small
- removed C8: 100nF-6.3V-0603, Capacitor_SMD:C_0603_1608Metric, symbol Device:C_Small
- removed J2: Power_In_Conn_01x02, Connector_PinHeader_2.54mm:PinHeader_1x02_P2.54mm_Vertical, symbol Connector_Generic:Conn_01x02
- removed R14: 1K1-1%-0603, Resistor_SMD:R_0603_1608Metric, symbol Device:R_Small
- removed R2: 4K7-0603, Resistor_SMD:R_0603_1608Metric, symbol Device:R_Small
- removed R9: 10K-0603, Resistor_SMD:R_0603_1608Metric, symbol Device:R_Small
- removed U3: ESP32-WROOM-32U, RF_Module:ESP32-WROOM-32U, symbol RF_Module:ESP32-WROOM-32U
- added C24: 100µF-6.3V-0603, Capacitor_SMD:C_0603_1608Metric, symbol Device:CP_Small
- added C5: 2µ2F-6.3V, Capacitor_SMD:C_0603_1608Metric, symbol Device:C_Small
- added C8: 330µF-50V, Capacitor_SMD:C_Elec_5x5.4, symbol Device:CP_Small
- added J4: USB_C_Receptacle_USB2.0, Connector_USB:USB_C_Receptacle_JAE_DX07S024WJ3R400, symbol Connector:USB_C_Receptacle_USB2.0
- added Q1, Q2: MMBT3904, Package_TO_SOT_SMD:SOT-23, symbol Transistor_BJT:MMBT3904
- added R15, R16, R17, R19: 10K-0603, Resistor_SMD:R_0603_1608Metric, symbol Device:R_Small
- added R18: 40K-0603, Resistor_SMD:R_0603_1608Metric, symbol Device:R_Small
- added U6: STUSB4500QTR, Package_DFN_QFN:QFN-24-1EP_4x4mm_P0.5mm_EP2.7x2.7mm, symbol Interface_USB:STUSB4500QTR
- added U7: ESP32-PICO-D4, Package_DFN_QFN:QFN-48-1EP_7x7mm_P0.5mm_EP5.3x5.3mm, symbol RF_Module:ESP32-PICO-D4
- C13: footprint Capacitor_SMD:C_0603_1608Metric -> Capacitor_SMD:C_0805_2012Metric
- C18: value 100nF-50V -> 100nF-25V; footprint Capacitor_SMD:C_0805_2012Metric -> Capacitor_SMD:C_0603_1608Metric
- C6: footprint Capacitor_SMD:C_0805_2012Metric -> Capacitor_SMD:C_0603_1608Metric
- C7: value 100nF-6.3V-0603 -> 2µ2F-6.3V
- D1: footprint LED_SMD:LED_Cree-PLCC4_2x2mm_CW -> Slimc_LED_SMD:WS2812_4020_SIDE
- J1: value Backpack_Conn_01x17 -> Backpack_Conn_02x09; footprint (none) -> Connector_PinSocket_2.54mm:PinSocket_2x09_P2.54mm_Vertical; symbol Connector:Screw_Terminal_01x17 -> Connector:Screw_Terminal_01x18
- R10: value 20K-0603 -> 4K7-0603
- R8: value 10K-0603 -> 4K7-0603
- U4: footprint Package_DFN_QFN:QFN-24-1EP_4x4mm_P0.5mm_EP2.6x2.6mm -> Package_SO:SOIC-8_3.9x4.9mm_P1.27mm
Connections:
- net ESP_RXD0 is gone; now on net VBUS: J1.17 (Pin_17)
- net GPIO12 is gone; now on net ESP_IO01: J1.7 (Pin_7)
- net GPIO4 is gone; now on net ESP_IO03: J1.5 (Pin_5)
- net GPIO5 is gone; now on net ESP_IO21: J1.6 (Pin_6)
- net +3V3: now also J1.2 (Pin_2), R3.2, U1.5 (VIO), U1.6 (VDD), C24.1, R15.1, U7.1 (VDDA), U7.19 (VDD3P3_RTC), U7.3 (VDDA3P3), U7.37 (VDD3P3_CPU), U7.4 (VDDA3P3), U7.43 (VDDA), U7.46 (VDDA); no longer R3.1
- net ESP_EN: now also J1.4 (Pin_4), R1.2, SW1.2, C5.2, Q1.3 (C), U7.9 (EN); no longer C7.1, R7.2, SW1.1
- net GND: now also C14.2, C15.2, C16.2, C17.2, C23.2, C7.2, J1.18 (Pin_18), SW1.1, U1.2 (GND), U1.25 (GND), C24.2, C5.1, C8.2, J4.A1 (GND), J4.A12 (GND), J4.B1 (GND), J4.B12 (GND), R19.2, U6.10 (GND), U6.25 (GND), U7.49 (GND); no longer C14.1, C15.1, C16.1, C17.1, J1.2 (Pin_2), SW1.2
- net VBUS: now also C8.1, J4.A4 (VBUS), J4.A9 (VBUS), J4.B4 (VBUS), J4.B9 (VBUS), R18.1, U6.24 (VDD)
- net at R4.2: now also D1.4 (DIN)
- net ESP_IO32: now reaches R4.1
- net ESP_IO32: now also U7.12 (IO32); no longer D1.4 (DIN)
- net ESP_IO00: now reaches J1.3 (Pin_3)
- net ESP_IO00: now also C7.1, R3.1, SW2.1, Q2.3 (C), U7.23 (IO0)
- net RTS: now reaches U1.19 (RTS)
- net RTS: now also Q2.2 (E), R16.1
- net ESP_IO03: now reaches U1.20 (RXD)
- net ESP_IO03: now also U7.40 (U0RXD/IO3)
- net ESP_IO01: now reaches U1.21 (TXD)
- net ESP_IO01: now also U7.41 (U0TXD/IO1)
- net DTR: now reaches U1.23 (DTR)
- net DTR: now also Q1.2 (E), R17.1
- net USB_D+: now reaches U1.3 (D+)
- net USB_D+: now also J4.A6 (D+), J4.B6 (D+)
- net USB_D-: now reaches U1.4 (D-)
- net USB_D-: now also J4.A7 (D-), J4.B7 (D-)
- net at U1.8 (VBUS): now also R18.2, R19.1
- net at U1.9 (~RSTb): now also R15.2
- net ESP_IO21: now reaches R8.2
- net ESP_IO21: now also U4.6 (SDA), U6.8 (SDA), U7.42 (IO21); no longer C7.2
- net AS5601_A renamed AS5601_ABI_A
- net AS5601_ABI_A: now also U7.36 (IO23)
- net AS5601_B renamed AS5601_ABI_B
- net AS5601_ABI_B: now also U7.14 (IO25)
- removed net ESP_IO0: R1.2, SW2.1
- net ESP_TXD0 renamed SVP
- net SVP: now also U7.5 (SENSOR_VP)
- net GPIO15 renamed ESP_IO22
- net ESP_IO22: now also R10.2, U4.7 (SCL), U6.7 (SCL), U7.39 (IO22)
- net GPIO19 renamed ESP_IO26
- net ESP_IO26: now also U7.15 (IO26)
- net GPIO26 renamed ESP_IO19
- net ESP_IO19: now also U7.38 (IO19)
- net GPIO33 renamed ESP_IO18
- net ESP_IO18: now also U7.35 (IO18)
- net GPIO34 renamed ESP_IO12
- net ESP_IO12: now also U7.18 (IO12)
- net GPIO35 renamed ESP_IO05
- net ESP_IO05: now also U7.34 (IO5)
- removed net I2C_SCL: J1.14 (Pin_14), R3.2, U4.7 (SCL)
- net I2C_SDA renamed SVN
- net SVN: now also U7.8 (SENSOR_VN); no longer U4.6 (SDA)
- removed net TMC2209_A1: C14.2, J3.2 (Pin_2), U5.24 (OA1)
- removed net TMC2209_A2: C15.2, J3.1 (Pin_1), U5.21 (OA2)
- removed net TMC2209_B1: C17.2, J3.3 (Pin_3), U5.26 (OB1)
- removed net TMC2209_B2: C16.2, J3.4 (Pin_4), U5.1 (OB2)
- net TMC2209_DIAG renamed ESP_IO02
- net ESP_IO02: now also U7.22 (IO2)
- net TMC2209_DIR renamed ESP_IO14
- net ESP_IO14: now also U7.17 (IO14)
- net TMC2209_EN renamed ESP_IO27
- net ESP_IO27: now also R7.2, U7.16 (IO27); no longer R10.2
- net TMC2209_STEP renamed ESP_IO13
- net ESP_IO13: now also U7.20 (IO13)
- net UART_RXD renamed ESP_IO17
- net UART_TXD renamed ESP_IO16
- new net: Q2.1 (B), R17.2
- new net: Q1.1 (B), R16.2
- new net ESP_IO04: J1.14 (Pin_14), U7.24 (IO4)
- new net ESP_IO09: U7.28 (SD2/IO9)
- new net ESP_IO10: U7.29 (SD3/IO10)
- new net ESP_IO15: U7.21 (IO15)
- new net ESP_IO33: U7.13 (IO33)
- new net ESP_IO34: U7.10 (IO34)
- new net ESP_IO35: U7.11 (IO35)
- new net ESP_LNA_IN: U7.2 (LNA_IN)
- new net TMC2209_OA1: C16.1, J3.3 (Pin_3), U5.24 (OA1)
- new net TMC2209_OA2: C17.1, J3.4 (Pin_4), U5.21 (OA2)
- new net TMC2209_OB1: C15.1, J3.2 (Pin_2), U5.26 (OB1)
- new net TMC2209_OB2: C14.1, J3.1 (Pin_1), U5.1 (OB2)
- new net USB_CC1: J4.A5 (CC1), U6.1 (CC1DB), U6.2 (CC1)
- new net USB_CC2: J4.B5 (CC2), U6.4 (CC2), U6.5 (CC2DB)
- no-connect marks 24 -> 29
Other:
- moved on the sheet: C1, C10, C11, C12, C18, C19, C2, C21, C22, C23, C3, C4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

Commit message: working on simplified design
Parts:
- removed C4: 22µF 6.3V, Capacitor_SMD:C_1206_3216Metric, symbol Device:CP_Small
- removed C5: 2µ2F-6.3V, Capacitor_SMD:C_0603_1608Metric, symbol Device:C_Small
- removed D2: B230A, Diode_SMD:D_1206_3216Metric, symbol Device:D_Schottky
- removed J4: USB_C_Receptacle_USB2.0, Connector_USB:USB_C_Receptacle_JAE_DX07S024WJ3R400, symbol Connector:USB_C_Receptacle_USB2.0
- removed L1: 4µ7H, Inductor_SMD:L_6.3x6.3_H3, symbol pspice:INDUCTOR
- removed R1: 4K7-0603, Resistor_SMD:R_0603_1608Metric, symbol Device:R_Small
- removed R5: 16K2-0603-1%, Resistor_SMD:R_0603_1608Metric, symbol Device:R_Small
- removed R6: 49K9-0603-1%, Resistor_SMD:R_0603_1608Metric, symbol Device:R_Small
- removed SW1: ESP_EN_SW_Push, Button_Switch_SMD:SW_SPST_B3U-1000P, symbol Switch:SW_Push
- removed U2: MP2360DG-LF, Package_DFN_QFN:TDFN-8-1EP_2x2mm_P0.5mm_EP0.8x1.2mm, symbol Slimc_Regulator_Switching:MP2360DG-LF
- added AE1: Antenna_Shield, symbol Device:Antenna_Shield
- added C20, C25: TBD, symbol Device:C_Small
- added C4: 10µF-0603, Capacitor_SMD:C_0603_1608Metric, symbol Device:C_Small
- added C?: 2µ2F-6.3V, Capacitor_SMD:C_0603_1608Metric, symbol Device:C_Small
- added J2: USB4120-03-C_REVA, Slimc_Connector_USB:GCT_USB4120-03-C_REVA, symbol Slimc_Connector_USB:USB4120-03-C_REVA
- added L1: TBD, symbol Device:L
- added R?: 4K7-0402, Resistor_SMD:R_0603_1608Metric, symbol Device:R_Small
- added SW?: ESP_EN_SW_Push, Button_Switch_SMD:SW_SPST_B3U-1000P, symbol Switch:SW_Push
- added U2: BD33FC0WEFJ-E2, Slimc_Converter_DCDC:BD33FC0WEFJ-E2, symbol Slimc_Converter_DCDC:BD33FC0WEFJ-E2
- C2: value 4µ7F 50V -> ??µF 35V
- C3: value 10nF-0603 -> ??µF-0603
- R10, R3, R8: value 4K7-0603 -> 4K7-0402
- R15: value 10K-0603 -> 10K-0402
- R4: value 230R-0603 -> 230R-0402
- R7: value 20K-0603 -> 20K-0402
- U5: digikey_part_number (none) -> 1460-1398-6-ND
Connections:
- net +3V3: now also C4.2, R?.2, U2.1 (VO)
- net ESP_EN: now also C?.1, R?.1, SW?.1
- net GND: now also C3.1, AE1.2 (Shield), C20.2, C25.1, C4.1, C?.2, J2.A1 (GND_A), J2.A12 (GND_A), J2.B1 (GND_B), J2.B12 (GND_B), J2.S1 (SHIELD), J2.S2 (SHIELD), J2.S3 (SHIELD), J2.S4 (SHIELD), SW?.2, U2.3 (GND)
- net USB_CC1: now also J2.A5 (CC1)
- net USB_CC2: now also J2.B5 (CC2)
- net USB_D+: now also J2.A6 (D1+), J2.B6 (D2+)
- net USB_D-: now also J2.A7 (D1-), J2.B7 (D2-)
- net VBUS: now also C3.2, J2.A4 (VBUS_A), J2.A9 (VBUS_A), J2.B4 (VBUS_B), J2.B9 (VBUS_B), U2.5 (EN), U2.8 (VCC)
- net DTR: no longer names the net of Q1.2 (E), R17.1, U1.23 (DTR)
- net ESP_LNA_IN: no longer names the net of U7.2 (LNA_IN)
- net ESP_LNA_IN: now also C20.1, L1.1
- net RTS: no longer names the net of Q2.2 (E), R16.1, U1.19 (RTS)
- new net: AE1.1 (A), C25.2, L1.2
- no-connect marks 29 -> 32
Other:
- moved on the sheet: C1, C10, C11, C12, C13, C14, C15, C16, C17, C18, C19, C21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
