File: circuits/driver-board.kicad_sch (KiCad schematic)
At the start: 76 parts, among them J1 Conn_01x18_Female, J2 USB4120-03-C_REVA, J3 Motor_Conn_01x04, J4 Screw_Terminals, J5 Conn_01x06_Female, Q1 SS8050-G, Q2 SS8050-G, SW1 RST_SW_Push, U1 CP2102N-A01-GQFN24, U2 BA33DD0T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

Commit message: gha
Parts:
- added R18, R19: 5.1K, Resistor_SMD:R_0402_1005Metric, symbol Device:R_Small
Connections:
- net GND: now also R18.1, R19.1
- net USB_CC2: now also R18.2, R19.2
- no-connect marks 32 -> 39
Other:
- note added: "Default sink config"
Changed lines of the file:
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@@
   (junction (at 59.055 223.52) (diameter 0) (color 0 0 0 0)
   )
+  (junction (at 41.91 88.9) (diameter 0) (color 0 0 0 0)
+  )
   (junction (at 417.195 180.34) (diameter 0) (color 0 0 0 0)
   )
@@
   (no_connect (at 43.18 170.18))
   (no_connect (at 76.835 256.54))
+  (no_connect (at 234.95 255.27))
+  (no_connect (at 234.95 247.65))
   (no_connect (at 73.66 160.02))
+  (no_connect (at 234.95 250.19))
   (no_connect (at 46.355 243.84))
   (no_connect (at 73.66 172.72))
@@
   (no_connect (at 46.355 241.3))
   (no_connect (at 297.18 215.9))
+  (no_connect (at 297.18 257.81))
   (no_connect (at 76.835 236.22))
   (no_connect (at 76.835 251.46))
@@
   (no_connect (at 63.5 134.62))
   (no_connect (at 215.9 63.5))
+  (no_connect (at 234.95 252.73))
   (no_connect (at 215.9 66.04))
   (no_connect (at 43.18 175.26))
@@
   (no_connect (at 76.835 246.38))
   (no_connect (at 73.66 170.18))
+  (no_connect (at 234.95 257.81))
   (no_connect (at 297.18 246.38))
   (no_connect (at 215.9 99.06))
@@
   (no_connect (at 73.66 149.86))
   (no_connect (at 215.9 101.6))
+  (no_connect (at 297.18 261.62))
   (wire (pts (xy 212.09 92.075) (xy 212.09 86.36))
     (stroke (width 0) (type default) (color 0 0 0 0))
@@
     (stroke (width 0) (type default) (color 0 0 0 0))
   )
+  (wire (pts (xy 40.64 86.36) (xy 40.64 88.9))
+    (stroke (width 0) (type default) (color 0 0 0 0))
+  )
   (wire (pts (xy 492.125 231.14) (xy 497.205 231.14))
     (stroke (width 0) (type default) (color 0 0 0 0))
@@
     (stroke (width 0) (type default) (color 0 0 0 0))
   )
+  (wire (pts (xy 43.18 88.9) (xy 43.18 86.36))
+    (stroke (width 0) (type default) (color 0 0 0 0))
+  )
   (wire (pts (xy 476.885 244.602) (xy 476.885 238.76))
     (stroke (width 0) (type default) (color 0 0 0 0))
@@
     (stroke (width 0) (type default) (color 0 0 0 0))
   )
+  (wire (pts (xy 40.64 88.9) (xy 41.91 88.9))
+    (stroke (width 0) (type default) (color 0 0 0 0))
+  )
   (wire (pts (xy 76.835 248.92) (xy 81.915 248.92))
     (stroke (width 0) (type default) (color 0 0 0 0))
@@
     (stroke (width 0) (type default) (color 0 0 0 0))
   )
+  (wire (pts (xy 43.18 73.66) (xy 43.18 81.28))
+    (stroke (width 0) (type default) (color 0 0 0 0))
+  )
   (wire (pts (xy 415.925 182.88) (xy 417.195 182.88))
     (stroke (width 0) (type default) (color 0 0 0 0))
   )
+  (wire (pts (xy 40.64 81.28) (xy 40.64 76.2))
+    (stroke (width 0) (type default) (color 0 0 0 0))
+  )
   (wire (pts (xy 463.55 116.84) (xy 463.55 124.46))
     (stroke (width 0) (type default) (color 0 0 0 0))
@@
     (stroke (width 0) (type default) (color 0 0 0 0))
   )
+  (wire (pts (xy 40.64 76.2) (xy 35.56 76.2))
+    (stroke (width 0) (type default) (color 0 0 0 0))
+  )
   (wire (pts (xy 134.62 278.765) (xy 134.62 277.495))
     (stroke (width 0) (type default) (color 0 0 0 0))
@@
     (stroke (width 0) (type default) (color 0 0 0 0))
   )
+  (wire (pts (xy 35.56 73.66) (xy 43.18 73.66))
+    (stroke (width 0) (type default) (color 0 0 0 0))
+  )
   (wire (pts (xy 359.41 278.13) (xy 367.03 278.13))
     (stroke (width 0) (type default) (color 0 0 0 0))
@@
     (stroke (width 0) (type default) (color 0 0 0 0))
   )
+  (wire (pts (xy 41.91 88.9) (xy 43.18 88.9))
+    (stroke (width 0) (type default) (color 0 0 0 0))
+  )
   (wire (pts (xy 259.715 107.95) (xy 259.715 101.6))
     (stroke (width 0) (type default) (color 0 0 0 0))
@@
     (stroke (width 0) (type default) (color 0 0 0 0))
   )
+  (wire (pts (xy 41.91 88.9) (xy 41.91 91.44))
+    (stroke (width 0) (type default) (color 0 0 0 0))
+  )
   (wire (pts (xy 269.24 104.14) (xy 264.16 104.14))
     (stroke (width 0) (type default) (color 0 0 0 0))
@@
     (effects (font (size 1.27 1.27) (thickness 0.254) bold italic) (justify left bottom))
   )
+  (text "Default\nsink config" (at 46.99 77.47 0)
+    (effects (font (size 1.27 1.27)) (justify left bottom))
+  )
   (text "POWER SUPPLY" (at 17.78 109.855 0)
     (effects (font (size 2.54 2.54) (thickness 0.508) bold) (justify left bottom))
@@
     )
   )
+  (global_label "USB_CC2" (shape input) (at 35.56 76.2 180) (fields_autoplaced)
+    (effects (font (size 1.27 1.27)) (justify right))
+    (property "Intersheet References" "${INTERSHEET_REFS}" (id 0) (at 116.84 128.27 0)
+      (effects (font (size 1.27 1.27)) hide)
+    )
+  )
   (global_label "ESP_IO10" (shape input) (at 229.87 226.06 180) (fields_autoplaced)
     (effects (font (size 1.27 1.27)) (justify right))
@@
     )
   )
+  (global_label "USB_CC2" (shape input) (at 35.56 73.66 180) (fields_autoplaced)
+    (effects (font (size 1.27 1.27)) (justify right))
+    (property "Intersheet References" "${INTERSHEET_REFS}" (id 0) (at 116.84 125.73 0)
+      (effects (font (size 1.27 1.27)) hide)
+    )
+  )
   (global_label "ESP_EN" (shape input) (at 138.43 260.985 0) (fields_autoplaced)
     (effects (font (size 1.27 1.27)) (justify left))
@@
     (pin "9")
   )
+  (symbol (lib_id "Device:R_Small") (at 40.64 83.82 0) (mirror x) (unit 1)
+    (in_bom yes) (on_board yes)
+    (property "Reference" "R18" (id 0) (at 36.83 85.09 0)
+      (effects (font (size 1.27 1.27)) (justify right))
+    )
+    (property "Value" "5.1K" (id 1) (at 38.735 82.55 0)
+      (effects (font (size 1.27 1.27)) (justify right))
+    )
+    (property "Footprint" "Resistor_SMD:R_0402_1005Metric" (id 2) (at 40.64 83.82 0)
+      (effects (font (size 1.27 1.27)) hide)
+    )
+    (property "Datasheet" "~" (id 3) (at 40.64 83.82 0)
+      (effects (font (size 1.27 1.27)) hide)
+    )
+    (pin "1")
+    (pin "2")
+  )
   (symbol (lib_id "Device:C_Small") (at 255.905 173.99 0) (mirror y) (unit 1)
     (in_bom yes) (on_board yes)
@@
     (pin "1")
   )
+  (symbol (lib_id "power:GND") (at 41.91 91.44 0) (unit 1)
+    (in_bom yes) (on_board yes)
+    (property "Reference" "#PWR041" (id 0) (at 41.91 97.79 0)
+      (effects (font (size 1.27 1.27)) hide)
+    )
+    (property "Value" "GND" (id 1) (at 42.037 95.8342 0))
+    (property "Footprint" "" (id 2) (at 41.91 91.44 0)
+      (effects (font (size 1.27 1.27)) hide)
+    )
+    (property "Datasheet" "" (id 3) (at 41.91 91.44 0)
+      (effects (font (size 1.27 1.27)) hide)
+    )
+    (pin "1")
+  )
   (symbol (lib_id "power:GND") (at 219.075 288.925 0) (unit 1)
     (in_bom yes) (on_board yes)
@@
     (pin "1")
   )
+  (symbol (lib_id "Device:R_Small") (at 43.18 83.82 180) (unit 1)
+    (in_bom yes) (on_board yes)
+    (property "Reference" "R19" (id 0) (at 46.99 85.09 0)
+      (effects (font (size 1.27 1.27)) (justify right))
+    )
+    (property "Value" "5.1K" (id 1) (at 45.085 82.55 0)
+      (effects (font (size 1.27 1.27)) (justify right))
+    )
+    (property "Footprint" "Resistor_SMD:R_0402_1005Metric" (id 2) (at 43.18 83.82 0)
+      (effects (font (size 1.27 1.27)) hide)
+    )
+    (property "Datasheet" "~" (id 3) (at 43.18 83.82 0)
+      (effects (font (size 1.27 1.27)) hide)
+    )
+    (pin "1")
+    (pin "2")
+  )
   (symbol (lib_id "power:GND") (at 233.68 288.29 0) (unit 1)
     (in_bom yes) (on_board yes)
@@
       (reference "#PWR040") (unit 1) (value "GND") (footprint "")
     )
+    (path "/a1eabea7-ac5a-4edb-8a93-eae2a0aa00a6"
+      (reference "#PWR041") (unit 1) (value "GND") (footprint "")
+    )
     (path "/00000000-0000-0000-0000-0000610e77fd"
       (reference "#PWR044") (unit 1) (value "GND") (footprint "")
@@
       (reference "R17") (unit 1) (value "10K") (footprint "Resistor_SMD:R_0402_1005Metric")
     )
+    (path "/6b887e5c-3cd4-49dc-806a-6820a4497130"
+      (reference "R18") (unit 1) (value "5.1K") (footprint "Resistor_SMD:R_0402_1005Metric")
+    )
+    (path "/ed8ff26a-9921-469f-9b6d-e78215c269ad"
+      (reference "R19") (unit 1) (value "5.1K") (footprint "Resistor_SMD:R_0402_1005Metric")
+    )
     (path "/00000000-0000-0000-0000-0000621debca"

Commit message: pcb layout redone
Parts:
- removed C18: 100nF, Capacitor_SMD:C_0402_1005Metric, symbol Device:CP_Small
- removed C19, C8: 330µF-50V, Capacitor_SMD:C_Elec_5x5.4, symbol Device:CP_Small
- removed R18, R19: 5.1K, Resistor_SMD:R_0402_1005Metric, symbol Device:R_Small
- removed TP1, TP2, TP3, TP4: TestPoint, symbol Connector:TestPoint
- removed U1: CP2102N-A01-GQFN24, Package_DFN_QFN:QFN-24-1EP_4x4mm_P0.5mm_EP2.6x2.6mm, symbol Interface_USB:CP2102N-A01-GQFN24
- added C14: 100nF, Capacitor_SMD:C_0402_1005Metric, symbol Device:C_Polarized_Small
- added C15, C8: 300µF-50V, Capacitor_SMD:C_Elec_5x5.4, symbol Device:C_Polarized_Small
- added R20, R21: 4K7, Resistor_SMD:R_0201_0603Metric, symbol Device:R_Small
- added U1: CP2102N-Axx-xQFN24, Package_DFN_QFN:QFN-24-1EP_4x4mm_P0.5mm_EP2.6x2.6mm, symbol Interface_USB:CP2102N-Axx-xQFN24
- C22, C23: now left out of the parts list
- R1, R11, R15, R2, R3, R4: footprint Resistor_SMD:R_0402_1005Metric -> Resistor_SMD:R_0201_0603Metric
- R10, R8: value 4K7 -> 5K1
Connections:
- net ESP_IO44 is gone; now on net UART0_RXD / ESP_IO44: J5.5 (Pin_5)
- net +3V3: now also C14.2, R20.1, R21.1, U1.5 (VIO), U1.6 (VDD), U1.8 (VBUS); no longer R10.1, R8.1
- net CP2102_DTR: now also U1.22 (~{DSR})
- net CP2102_RTS: now also U1.19 (~{RTS})
- net ESP_IO09: no longer U8.5, U8.7
- net ESP_IO10: no longer R3.2, U8.6
- net GND: now also R10.2, R8.2, C14.1, C15.2, C8.2, U1.2 (GND), U1.25 (GND)
- net USB_CC1: now also R8.1
- net USB_CC2: now also R10.1
- net USB_D+: now also U1.3 (D+); no longer U3.26 (GPIO20/USB_D+/ADC2_CH9)
- net USB_D-: now also U1.4 (D-); no longer U3.25 (GPIO19/USB_D-/ADC2_CH8)
- net VBUS: now also C15.1, C8.1
- net at R15.2: now also U1.9 (~{RST})
- net ESP_IO47: now reaches C27.2, R14.2, U3.37 (SPICLK_P/GPIO47)
- net UART0_RXD / ESP_IO44: now reaches U3.50 (U0RXD/PROG/GPIO44)
- net UART0_RXD / ESP_IO44: now also U1.20 (RXD)
- net AS5601_ABI_A renamed AS5601_A_ITR / ESP_IO11
- net AS5601_ABI_B renamed AS5601_B_ITR / ESP_IO12
- net ESP_IO01 renamed LED / ESP_IO01
- net ESP_IO04 renamed I2C_SCL / ESP_IO04
- net I2C_SCL / ESP_IO04: now also R20.2; no longer R10.2
- net ESP_IO05 renamed I2C_SDA / ESP_IO05
- net I2C_SDA / ESP_IO05: now also R21.2; no longer R8.2
- net ESP_IO06 renamed TMC2209_EN / ESP_IO06
- net ESP_IO07 renamed TMC2209_STEP / ESP_IO07
- net ESP_IO08 renamed TMC2209_DIR / ESP_IO08
- net ESP_IO19 renamed USB_D- / ESP_IO19
- net USB_D- / ESP_IO19: now also U3.25 (GPIO19/USB_D-/ADC2_CH8)
- net ESP_IO43 renamed UART0_TXD / ESP_IO43
- net UART0_TXD / ESP_IO43: now also U1.21 (TXD)
- net ESP_IO45 renamed UART1_TXD / ESP_IO45
- net ESP_IO46 renamed UART1_RXD / ESP_IO46
- net ESP_SPICLK renamed SPICLK / ESP_IO30
- net ESP_SPICS1 renamed SPICS1 / ESP_IO26
- net ESP_SPID renamed SPID / ESP_IO32
- net ESP_SPIHD renamed SPIHD / ESP_IO27
- net ESP_SPIQ renamed SPIQ / ESP_IO31
- net ESP_SPIWP renamed SPIWP / ESP_IO28
- net ESP_XTAL_N renamed XTAL_N
- net ESP_XTAL_P renamed XTAL_P
- net TMC2209_OA1: no longer names the net of U5.24 (OA1)
- net TMC2209_OA1: now also J3.2 (Pin_2); no longer J3.3 (Pin_3)
- net TMC2209_OA2: no longer names the net of J3.4 (Pin_4)
- net TMC2209_OA2: now also U5.1 (OB2); no longer U5.21 (OA2)
- net TMC2209_OB1: no longer names the net of U5.26 (OB1)
- net TMC2209_OB1: now also J3.3 (Pin_3); no longer J3.2 (Pin_2)
- net TMC2209_OB2: no longer names the net of J3.1 (Pin_1)
- net TMC2209_OB2: now also U5.21 (OA2); no longer U5.1 (OB2)
- new net SR_Q / ESP_IO09: U8.5, U8.7
- new net SR_S / ESP_IO10: R3.2, U8.6
- new net USB_D+ / ESP_IO20: U3.26 (GPIO20/USB_D+/ADC2_CH9)
- no-connect marks 39 -> 48
Other:
- note added: "Delay boot ~50µs"
- note added: "INTERRUPTS"
- note removed: "Default sink config"
- note removed: "Delay boot ~50µS"
- moved on the sheet: AE1, C1, C10, C11, C12, C13, C2, C20, C21, C22, C23, C25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

Commit message: adjusted tmc2209 circuitry and redid overall comp placement
Parts:
- removed C15, C8: 300µF-50V, Capacitor_SMD:C_Elec_5x5.4, symbol Device:C_Polarized_Small
- removed C21: 100nF-50V, Capacitor_SMD:C_0402_1005Metric, symbol Device:C_Small
- removed C22, C23: 10µF-50V, Capacitor_SMD:C_2220_5650Metric, symbol Device:C_Small
- added C15, C16: 10µF-50V, Capacitor_SMD:C_1210_3225Metric, symbol Device:C_Small
- added C8: 1µF-50V, Capacitor_SMD:C_0603_1608Metric, symbol Device:C_Small
- added R18: 20K, Resistor_SMD:R_0402_1005Metric, symbol Device:R_Small
- added R19: 100K, Resistor_SMD:R_0201_0603Metric, symbol Device:R_Small
- C10, C14, C9: footprint Capacitor_SMD:C_0402_1005Metric -> Capacitor_SMD:C_0603_1608Metric
- C11: value 22nF-50V-0603 -> 22nF-50V; footprint Capacitor_SMD:C_0402_1005Metric -> Capacitor_SMD:C_0805_2012Metric
- C12, C13: value 100nF -> 100nF-50V; footprint Capacitor_SMD:C_0805_2012Metric -> Capacitor_SMD:C_0603_1608Metric
- R12, R13: value 0R11-0805-1W -> 0R100; footprint Resistor_SMD:R_0805_2012Metric -> Resistor_SMD:R_2010_5025Metric
- R2: footprint Resistor_SMD:R_0201_0603Metric -> Resistor_SMD:R_0402_1005Metric
- R3: value 20K -> 0R100-0603; footprint Resistor_SMD:R_0201_0603Metric -> Resistor_SMD:R_0603_1608Metric
- U5: footprint Package_SO:HTSSOP-28-1EP_4.4x9.7mm_P0.65mm_EP3.4x9.5mm_ThermalVias -> Package_DFN_QFN:QFN-28-1EP_5x5mm_P0.5mm_EP3.35x3.35mm_ThermalVias
Connections:
- net +3V3: now also R2.1; no longer R3.1
- net GND: now also R3.2, C15.2, C16.2, R18.2, R19.2; no longer R2.2, U5.20 (STDBY)
- net SR_S / ESP_IO10: now also R2.2, R18.1; no longer R3.2
- net TMC2209_DIAG: no longer R2.1
- net VBUS: now also C12.1, C13.1, C15.1, C16.1, C8.1
- net at R12.2, U5.23 (BRA): no longer C12.1
- net at R13.2, U5.27 (BRB): no longer C13.1
- net TMC2209_OB2: now reaches J3.4 (Pin_4), U5.1 (OB2)
- net TMC2209_OA2: now reaches J3.1 (Pin_1), U5.21 (OA2)
- net TMC2209_OA1: now reaches J3.2 (Pin_2), U5.24 (OA1)
- net TMC2209_OB1: now reaches J3.3 (Pin_3), U5.26 (OB1)
- net XTAL_N: no longer names the net of C26.2, U3.53 (XTAL_N), Y1.3
- net XTAL_P: no longer names the net of C35.2, U3.54 (XTAL_P), Y1.1
- new net: R19.1, U5.20 (STDBY)
- new net: C8.2, R3.1
Other:
- note added: "(RSA,RSB) = 2010 1W"
- note added: "PULL TO BE DETERMINED"
- note added: "STRPPING POWER PINS"
- note added: "Source sensing"
- note added: "from https://www.digikey.at/en/products/detail/trinamic-motion-control-gmbh/TMC2209-BOB/10490037"
- moved on the sheet: C26, C27, C35, D3, J2, J3, J4, R14, R2, R5, R6, R7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
