File: circuits-proto/driver-board.kicad_sch (KiCad schematic)
At the start: 75 parts, among them J1 Conn_01x18_Female, J2 USB4120-03-C_REVA, J3 Motor_Conn_01x04, J4 Screw_Terminals, J5 Conn_01x06_Female, Q1 SS8050-G, Q2 SS8050-G, SW1 RST_SW_Push, U1 CP2102N-Axx-xQFN24, U2 BA033CC0FP-E2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

Commit message: updated library paths
Parts:
- removed J2: USB4120-03-C_REVA, Slimc_Connector_USB:GCT_USB4120-03-C_REVA, symbol Slimc_Connector_USB:USB4120-03-C_REVA
- removed Q1, Q2: SS8050-G, Package_TO_SOT_SMD:SOT-23, symbol Device:Q_NPN_BEC
- removed R15: 10K, Resistor_SMD:R_0201_0603Metric, symbol Device:R_Small
- removed R16, R17: 10K, Resistor_SMD:R_0402_1005Metric, symbol Device:R_Small
- removed U1: CP2102N-Axx-xQFN24, Package_DFN_QFN:QFN-24-1EP_4x4mm_P0.5mm_EP2.6x2.6mm, symbol Interface_USB:CP2102N-Axx-xQFN24
- removed U6: STUSB4500QTR, Package_DFN_QFN:QFN-24-1EP_4x4mm_P0.5mm_EP2.7x2.7mm, symbol Interface_USB:STUSB4500QTR
Connections:
- no-connect marks 56 -> 29
Other:
- note removed: "LET STUSB4500 enable BA33DD0T?"
- note removed: "Program Sequence DTR RTS --> EN IO00 1 1 1 1 0 0 1 1 1 0 0 1 0 1 1 0"
- note removed: "from https://dl.espressif.com/dl/SCH_ESP32-S3-DEVKITC-1_V1_20210312C.pdf"
